Commit message: added egh gripper

File: rbkairos_description/robots/rbkairos_ur10.urdf.xacro (robot description, xacro)
@@ -9,4 +9,6 @@
     <!-- Include UR-10 ARM -->
 	<xacro:include filename="$(find ur_description)/urdf/ur10.urdf.xacro" />
+	<!-- Include EGH  -->
+	<xacro:include filename="$(find egh_gripper_support)/urdf/egh_gripper.urdf.xacro" />
   	<!-- Import summit XL wheels -->
   	<xacro:include filename="$(find summit_xl_description)/urdf/wheels/omni_wheel.urdf.xacro" />
@@ -112,4 +114,8 @@
   			<origin xyz="${front_rgbd_camera_offset_x} ${front_rgbd_camera_offset_y} ${front_rgbd_camera_offset_z}" rpy="0 0 0"/>
   		</xacro:sensor_zed-->
+		<!-- Schunk EGH -->
+		<xacro:egh_gripper prefix="$(arg prefix)egh_gripper" parent="$(arg prefix)arm_tool0">
+			<origin xyz="0.0 0.0 0.0" rpy="0 -${pi/2} 0"/>
+		</xacro:egh_gripper>
     </xacro:macro>
     <!-- Gazebo ros control pluggins -->

Commit message: fixed arm rotation

File: rbkairos_description/robots/rbkairos_ur10.urdf.xacro (robot description, xacro)
@@ -53,5 +53,5 @@
     <xacro:property name="arm_orientation_r" value="0"/>
     <xacro:property name="arm_orientation_p" value="0"/>
-    <xacro:property name="arm_orientation_y" value="0"/>
+    <xacro:property name="arm_orientation_y" value="${pi}"/>
     <xacro:macro name="rbkairos" params="prefix publish_bf hq load_kinematics_file">
   		<!-- *************** -->
